File: EAGLE_Files/Confundus.brd (EAGLE design)
At the start: 43.8 x 20 mm, 91 parts, among them IC2 ATTINY1616-MNR, IC4 TPS61291DRVT, J5 SM03B-SRSS-TB_LF__SN_, Q3 DMG3415U-7, SW1 MLL1200S

Commit message: Adjustement to the charging circuit
Other:
- board text added: "Again and Again"
- board text added: "Confundus v1.1 by Tanmoy"
- board text removed: "Confundus v1.0 by Tanmoy"
- board text removed: "To the moon and back"
