File: EAGLE_Files/Confundus.sch (EAGLE design)
At the start: 91 parts, among them IC2 ATTINY1616-MNR, IC4 TPS61291DRVT, J5 SM03B-SRSS-TB_LF__SN_, Q3 DMG3415U-7, SW1 MLL1200S

Commit message: Adjustement to the charging circuit
Other:
- note added: "LED Matrix"
- note added: "This is a charging circuit for a LIC Super Capacitor. It is combined with a 3.3V buck converter to power an ATTiny1616 Microcontroller."
Changed lines of the file:
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@@
 <sheet>
 <plain>
+<text x="165.1" y="-182.88" size="1.778" layer="94">LED Matrix</text>
+<text x="165.1" y="10.16" size="1.778" layer="94">This is a charging circuit for a LIC Super
+Capacitor. It is combined with a 3.3V
+buck converter to power an ATTiny1616
+ Microcontroller.</text>
 </plain>
 <instances>
@@
 </drawing>
 <compatibility>
+<note version="6.3" minversion="6.2.2" severity="warning">
+Since Version 6.2.2 text objects can contain more than one line,
+which will not be processed correctly with this version.
+</note>
 <note version="8.2" severity="warning">
 Since Version 8.2, EAGLE supports online libraries. The ids
