File: EAGLE_Files/ConfundusV2.sch (EAGLE design)
At the start: 89 parts, among them IC1 MIC5219YM5_TR, IC2 ATTINY1616-MNR, IC4 TPS61291DRVT, J5 SM03B-SRSS-TB_LF__SN_, Q1 DMG3415U-7, Q3 DMG3415U-7, SW1 MLL1200S

Commit message: Updating the circuit adjustments for introduction of a Schottky diode
Parts:
- removed Q1: DMG3415U-7, DMG3415U-7:DMG3415U-7
- added D1: MBR120VLSFT1G, MBR120VLSFT1G:MBR120VLSFT1G
Connections:
- net GND: no longer Q1.G
- net N$10: now also D1.A; no longer Q1.S
- net N$12: now also D1.K; no longer Q1.D
Changed lines of the file:
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@@
 <part name="FRAME3" library="frames" library_urn="urn:adsk.eagle:library:229" deviceset="A4L-LOC" device=""/>
 <part name="IC1" library="MIC5219YM5_TR" deviceset="MIC5219YM5_TR" device="" override_package3d_urn="urn:adsk.eagle:package:52775026/2" override_package_urn="urn:adsk.eagle:footprint:52775027/1"/>
-<part name="Q1" library="DMG3415U-7" deviceset="DMG3415U-7" device="" override_package3d_urn="urn:adsk.eagle:package:51305947/2" override_package_urn="urn:adsk.eagle:footprint:51305948/1"/>
 <part name="U$3" library="Adafruit Feather STM32F405 Express" deviceset="MICROBUILDER_VBUS" device="" value="VBUS"/>
 <part name="U$7" library="Adafruit Feather STM32F405 Express" deviceset="MICROBUILDER_VBUS" device="" value="VBUS"/>
 <part name="R4" library="ERJ1TYJ220U" deviceset="ERJ1TYJ220U" device="" override_package3d_urn="urn:adsk.eagle:package:52775042/2" override_package_urn="urn:adsk.eagle:footprint:52775043/1"/>
+<part name="D1" library="MBR120VLSFT1G" deviceset="MBR120VLSFT1G" device="" override_package3d_urn="urn:adsk.eagle:package:53013620/2" override_package_urn="urn:adsk.eagle:footprint:53013621/1"/>
 </parts>
 <sheets>
@@
 <attribute name="VALUE" x="125.73" y="160.02" size="1.778" layer="96" align="center-left"/>
 </instance>
-<instance part="Q1" gate="G$1" x="170.18" y="160.02" smashed="yes" rot="R270" grouprefs="ADJUSTABLE_LDO">
-<attribute name="NAME" x="166.37" y="148.59" size="1.778" layer="95" align="center-left"/>
-<attribute name="VALUE" x="171.45" y="158.75" size="1.778" layer="96" align="center-left"/>
-</instance>
 <instance part="U$3" gate="G$1" x="111.76" y="162.56" smashed="yes" grouprefs="ADJUSTABLE_LDO">
 <attribute name="VALUE" x="110.236" y="163.576" size="1.27" layer="96"/>
@@
 <attribute name="NAME" x="189.23" y="135.89" size="1.778" layer="95" rot="R270" align="center-left"/>
 <attribute name="VALUE" x="186.69" y="148.59" size="1.778" layer="96" rot="R270" align="center-left"/>
+</instance>
+<instance part="D1" gate="G$1" x="180.34" y="152.4" smashed="yes" rot="R180" grouprefs="ADJUSTABLE_LDO">
+<attribute name="NAME" x="173.99" y="147.32" size="1.778" layer="95" rot="R180" align="center-left"/>
+<attribute name="VALUE" x="181.61" y="157.48" size="1.778" layer="96" rot="R180" align="center-left"/>
 </instance>
 </instances>
@@
 <pinref part="R2" gate="G$1" pin="1"/>
 <wire x1="160.02" y1="121.92" x2="160.02" y2="124.46" width="0.1524" layer="91" grouprefs="ADJUSTABLE_LDO"/>
-<pinref part="Q1" gate="G$1" pin="G"/>
-<wire x1="170.18" y1="160.02" x2="170.18" y2="162.56" width="0.1524" layer="91" grouprefs="ADJUSTABLE_LDO"/>
-<wire x1="170.18" y1="162.56" x2="165.1" y2="162.56" width="0.1524" layer="91" grouprefs="ADJUSTABLE_LDO"/>
-<wire x1="165.1" y1="162.56" x2="165.1" y2="121.92" width="0.1524" layer="91" grouprefs="ADJUSTABLE_LDO"/>
-<wire x1="165.1" y1="121.92" x2="160.02" y2="121.92" width="0.1524" layer="91" grouprefs="ADJUSTABLE_LDO"/>
-<junction x="160.02" y="121.92" grouprefs="ADJUSTABLE_LDO"/>
 </segment>
 <segment>
@@
 <wire x1="149.86" y1="152.4" x2="149.86" y2="144.78" width="0.1524" layer="91" grouprefs="ADJUSTABLE_LDO"/>
 <pinref part="C10" gate="G$1" pin="1"/>
-<pinref part="Q1" gate="G$1" pin="S"/>
 <wire x1="149.86" y1="152.4" x2="160.02" y2="152.4" width="0.1524" layer="91" grouprefs="ADJUSTABLE_LDO"/>
 <junction x="149.86" y="152.4" grouprefs="ADJUSTABLE_LDO"/>
@@
 <wire x1="160.02" y1="149.86" x2="160.02" y2="152.4" width="0.1524" layer="91" grouprefs="ADJUSTABLE_LDO"/>
 <junction x="160.02" y="152.4" grouprefs="ADJUSTABLE_LDO"/>
+<pinref part="D1" gate="G$1" pin="A"/>
 </segment>
 </net>
 <net name="N$12" class="0">
 <segment>
-<pinref part="Q1" gate="G$1" pin="D"/>
-<wire x1="180.34" y1="152.4" x2="182.88" y2="152.4" width="0.1524" layer="91" grouprefs="ADJUSTABLE_LDO"/>
 <pinref part="R4" gate="G$1" pin="1"/>
 <wire x1="182.88" y1="152.4" x2="182.88" y2="149.86" width="0.1524" layer="91" grouprefs="ADJUSTABLE_LDO"/>
-</segment>
-</net>
+<pinref part="D1" gate="G$1" pin="K"/>
+<wire x1="180.34" y1="152.4" x2="182.88" y2="152.4" width="0.1524" layer="91" grouprefs="ADJUSTABLE_LDO"/>
+</segment>
+</net>
